File: NodeMcuDevKitV1.sch (KiCad schematic (older format))
At the start: 23 parts, among them Q1 S8050, Q2 S8050, U1 ESP-12E, U2 CP2102, U3 NCP1117-3.3_SOT223, U4 USB_Micro_5S_B

Commit message: 2019/03/19 - Complete Schematics
Parts:
- added D1: LED, symbol Device:LED
- added J1, J2: Conn_01x15_Female, symbol Connector:Conn_01x15_Female
- added R10: 0 (NC), symbol Device:R
- added R11, R12, R9: 470, symbol Device:R
- added R13: 220k (1%), symbol Device:R
- added R14: 100k (1%), symbol Device:R
- added SW1: KEY_RST, symbol Switch:SW_SPST
- added SW2: KEY_FLASH, symbol Switch:SW_SPST
- renumbered D1 to D2, U4 to U3, U3 to U4
Connections:
- net labels added: ADC_EX, RESV
- wire segments 124 -> 179
Other:
- note added: "ADC"
- note added: "IO Conn"
- note added: "Key"
- note added: "Use 1% resistors here"
- note added: "Use this resistor\nin sleep mode only."
- moved on the sheet: C1, C2, C3, C4, C5, C6, C7, C8, D2, Q1, Q2, R1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

Commit message: 2019/03/19 - Add PCB and Autorouting
Parts:
- C1, C3, C4, C5, C6, C8: footprint (none) -> Capacitor_SMD:C_0402_1005Metric
- C2: footprint (none) -> Capacitor_Tantalum_SMD:CP_EIA-3528-21_Kemet-B
- C7: footprint (none) -> Capacitor_SMD:C_0805_2012Metric
- D1: footprint (none) -> LED_SMD:LED_0603_1608Metric
- D2: footprint Diode_THT:D_DO-41_SOD81_P10.16mm_Horizontal -> Diode_SMD:D_0805_2012Metric
- J1: footprint (none) -> Connector_PinSocket_2.54mm:PinSocket_1x15_P2.54mm_Vertical
- J2: footprint (none) -> Connector_PinHeader_2.54mm:PinHeader_1x15_P2.54mm_Vertical
- Q1, Q2: footprint Package_TO_SOT_THT:TO-92_Inline -> digikey-footprints:SOT-23-3
- R1, R10, R11, R12, R13, R14, R2, R3, R4, R5, R6, R7, R8, R9: footprint (none) -> Resistor_SMD:R_0402_1005Metric
- SW1, SW2: footprint (none) -> Button_Switch_SMD:SW_SPST_PTS810
- U1: footprint (none) -> RF_Module:ESP-12E
- U2: footprint (none) -> Package_DFN_QFN:QFN-28-1EP_5x5mm_P0.5mm_EP3.35x3.35mm
- U3: footprint (none) -> digikey-footprints:USB_Micro_B_Female_10118192
Changed lines of the file:
@@
 F 0 "R1" V 1300 1950 50  0000 C CNN
 F 1 "12k" V 1300 2300 50  0000 C CNN
-F 2 "" V 1280 2100 50  0001 C CNN
+F 2 "Resistor_SMD:R_0402_1005Metric" V 1280 2100 50  0001 C CNN
 F 3 "~" H 1350 2100 50  0001 C CNN
 	1    1350 2100
@@
 F 0 "R2" V 1300 2150 50  0000 C CNN
 F 1 "12k" V 1300 2500 50  0000 C CNN
-F 2 "" V 1280 2300 50  0001 C CNN
+F 2 "Resistor_SMD:R_0402_1005Metric" V 1280 2300 50  0001 C CNN
 F 3 "~" H 1350 2300 50  0001 C CNN
 	1    1350 2300
@@
 F 0 "R3" V 1300 2350 50  0000 C CNN
 F 1 "12k" V 1300 2700 50  0000 C CNN
-F 2 "" V 1280 2500 50  0001 C CNN
+F 2 "Resistor_SMD:R_0402_1005Metric" V 1280 2500 50  0001 C CNN
 F 3 "~" H 1350 2500 50  0001 C CNN
 	1    1350 2500
@@
 F 0 "R4" V 1300 2550 50  0000 C CNN
 F 1 "12k" V 1300 2900 50  0000 C CNN
-F 2 "" V 1280 2700 50  0001 C CNN
+F 2 "Resistor_SMD:R_0402_1005Metric" V 1280 2700 50  0001 C CNN
 F 3 "~" H 1350 2700 50  0001 C CNN
 	1    1350 2700
@@
 F 0 "R5" V 1300 2750 50  0000 C CNN
 F 1 "12k" V 1300 3100 50  0000 C CNN
-F 2 "" V 1280 2900 50  0001 C CNN
+F 2 "Resistor_SMD:R_0402_1005Metric" V 1280 2900 50  0001 C CNN
 F 3 "~" H 1350 2900 50  0001 C CNN
 	1    1350 2900
@@
 F 0 "C1" H 2250 2950 50  0000 L CNN
 F 1 "100nF" H 2250 2750 50  0000 L CNN
-F 2 "" H 2238 2700 50  0001 C CNN
+F 2 "Capacitor_SMD:C_0402_1005Metric" H 2238 2700 50  0001 C CNN
 F 3 "~" H 2200 2850 50  0001 C CNN
 	1    2200 2850
@@
 F 0 "C2" H 2850 2600 50  0000 L CNN
 F 1 "100uF" H 2700 2400 50  0000 L CNN
-F 2 "" H 2800 2500 50  0001 C CNN
+F 2 "Capacitor_Tantalum_SMD:CP_EIA-3528-21_Kemet-B" H 2800 2500 50  0001 C CNN
 F 3 "~" H 2800 2500 50  0001 C CNN
 	1    2800 2500
@@
 F 0 "U1" H 2000 4900 50  0000 C CNN
 F 1 "ESP-12E" H 2000 4800 50  0000 C CNN
-F 2 "" H 2000 4600 50  0001 C CNN
+F 2 "RF_Module:ESP-12E" H 2000 4600 50  0001 C CNN
 F 3 "" H 2000 4600 50  0001 C CNN
 	1    2000 4600
@@
 F 0 "U2" H 5100 3600 50  0000 C CNN
 F 1 "CP2102" H 5100 3500 50  0000 C CNN
-F 2 "" H 4600 2600 50  0001 C CNN
+F 2 "Package_DFN_QFN:QFN-28-1EP_5x5mm_P0.5mm_EP3.35x3.35mm" H 4600 2600 50  0001 C CNN
 F 3 "" H 4600 2600 50  0001 C CNN
 	1    5100 3300
@@
 F 0 "C5" V 5200 1750 50  0000 L CNN
 F 1 "10uF" V 5100 1800 50  0000 L CNN
-F 2 "" H 5288 1750 50  0001 C CNN
+F 2 "Capacitor_SMD:C_0402_1005Metric" H 5288 1750 50  0001 C CNN
 F 3 "~" H 5250 1900 50  0001 C CNN
 	1    5250 1900
@@
 F 0 "C3" H 3600 2950 50  0000 L CNN
 F 1 "10uF" H 3525 3150 50  0000 L CNN
-F 2 "" H 3638 2900 50  0001 C CNN
+F 2 "Capacitor_SMD:C_0402_1005Metric" H 3638 2900 50  0001 C CNN
 F 3 "~" H 3600 3050 50  0001 C CNN
 	1    3600 3050
@@
 F 0 "C4" H 3850 2950 50  0000 C CNN
 F 1 "100nF" H 3775 3150 50  0000 C CNN
-F 2 "" H 3838 2900 50  0001 C CNN
+F 2 "Capacitor_SMD:C_0402_1005Metric" H 3838 2900 50  0001 C CNN
 F 3 "~" H 3800 3050 50  0001 C CNN
 	1    3800 3050
@@
 F 0 "R8" V 4000 3650 50  0000 C CNN
 F 1 "470" V 4000 4000 50  0000 C CNN
-F 2 "" V 3980 3800 50  0001 C CNN
+F 2 "Resistor_SMD:R_0402_1005Metric" V 3980 3800 50  0001 C CNN
 F 3 "~" H 4050 3800 50  0001 C CNN
 	1    4050 3800
@@
 F 0 "C6" V 5300 2200 50  0000 C CNN
 F 1 "100nF" V 5100 2100 50  0000 C CNN
-F 2 "" H 5288 1950 50  0001 C CNN
+F 2 "Capacitor_SMD:C_0402_1005Metric" H 5288 1950 50  0001 C CNN
 F 3 "~" H 5250 2100 50  0001 C CNN
 	1    5250 2100
@@
 F 0 "Q1" H 3625 4075 50  0000 L CNN
 F 1 "S8050" H 3475 4150 50  0000 L CNN
-F 2 "Package_TO_SOT_THT:TO-92_Inline" H 3900 4225 50  0001 L CIN
+F 2 "digikey-footprints:SOT-23-3" H 3900 4225 50  0001 L CIN
 F 3 "http://www.unisonic.com.tw/datasheet/S8050.pdf" H 3700 4300 50  0001 L CNN
 	1    3700 4300
@@
 F 0 "Q2" H 3625 5175 50  0000 L CNN
 F 1 "S8050" H 3475 5250 50  0000 L CNN
-F 2 "Package_TO_SOT_THT:TO-92_Inline" H 3900 5325 50  0001 L CIN
+F 2 "digikey-footprints:SOT-23-3" H 3900 5325 50  0001 L CIN
 F 3 "http://www.unisonic.com.tw/datasheet/S8050.pdf" H 3700 5400 50  0001 L CNN
 	1    3700 5400
@@
 F 0 "R6" H 3925 4400 50  0000 C CNN
 F 1 "12k" H 3875 4550 50  0000 C CNN
-F 2 "" V 3930 4550 50  0001 C CNN
+F 2 "Resistor_SMD:R_0402_1005Metric" V 3930 4550 50  0001 C CNN
 F 3 "~" H 4000 4550 50  0001 C CNN
 	1    4000 4550
@@
 F 0 "R7" H 3925 5000 50  0000 C CNN
 F 1 "12k" H 3875 5150 50  0000 C CNN
-F 2 "" V 3930 5150 50  0001 C CNN
+F 2 "Resistor_SMD:R_0402_1005Metric" V 3930 5150 50  0001 C CNN
 F 3 "~" H 4000 5150 50  0001 C CNN
 	1    4000 5150
@@
 F 0 "U3" H 5100 5463 50  0000 C CNN
 F 1 "USB_Micro_5S_B" H 5100 5373 50  0000 C CNN
-F 2 "" H 5000 5000 50  0001 C CNN
+F 2 "digikey-footprints:USB_Micro_B_Female_10118192" H 5000 5000 50  0001 C CNN
 F 3 "" H 5000 5000 50  0001 C CNN
 	1    5100 5000
@@
 F 0 "D2" H 7200 2600 50  0000 C CNN
 F 1 "1N5819" H 7200 2825 50  0000 C CNN
-F 2 "Diode_THT:D_DO-41_SOD81_P10.16mm_Horizontal" H 7200 2525 50  0001 C CNN
+F 2 "Diode_SMD:D_0805_2012Metric" H 7200 2525 50  0001 C CNN
 F 3 "http://www.vishay.com/docs/88525/1n5817.pdf" H 7200 2700 50  0001 C CNN
 	1    7200 2700
@@
 F 0 "C7" H 6575 2350 50  0000 L CNN
 F 1 "10uF 25V" H 6500 2150 50  0000 L CNN
-F 2 "" H 6738 2100 50  0001 C CNN
+F 2 "Capacitor_SMD:C_0805_2012Metric" H 6738 2100 50  0001 C CNN
 F 3 "~" H 6700 2250 50  0001 C CNN
 	1    6700 2250
@@
 F 0 "C8" H 7575 2350 50  0000 L CNN
 F 1 "10uF" H 7500 2175 50  0000 L CNN
-F 2 "" H 7738 2100 50  0001 C CNN
+F 2 "Capacitor_SMD:C_0402_1005Metric" H 7738 2100 50  0001 C CNN
 F 3 "~" H 7700 2250 50  0001 C CNN
 	1    7700 2250
@@
 F 0 "J1" H 9250 3550 50  0000 L CNN
 F 1 "Conn_01x15_Female" V 9650 2325 50  0000 L CNN
-F 2 "" H 9600 2700 50  0001 C CNN
+F 2 "Connector_PinSocket_2.54mm:PinSocket_1x15_P2.54mm_Vertical" H 9600 2700 50  0001 C CNN
 F 3 "~" H 9600 2700 50  0001 C CNN
 	1    9600 2700
@@
 F 0 "J2" H 9700 3550 50  0000 C CNN
 F 1 "Conn_01x15_Female" V 10050 2700 50  0000 C CNN
-F 2 "" H 10000 2700 50  0001 C CNN
+F 2 "Connector_PinHeader_2.54mm:PinHeader_1x15_P2.54mm_Vertical" H 10000 2700 50  0001 C CNN
 F 3 "~" H 10000 2700 50  0001 C CNN
 	1    10000 2700
@@
 F 0 "R9" H 6670 3995 50  0000 L CNN
 F 1 "470" H 6670 3905 50  0000 L CNN
-F 2 "" V 6530 3950 50  0001 C CNN
+F 2 "Resistor_SMD:R_0402_1005Metric" V 6530 3950 50  0001 C CNN
 F 3 "~" H 6600 3950 50  0001 C CNN
 	1    6600 3950
@@
 F 0 "R10" H 6670 4895 50  0000 L CNN
 F 1 "0 (NC)" H 6670 4805 50  0000 L CNN
-F 2 "" V 6530 4850 50  0001 C CNN
+F 2 "Resistor_SMD:R_0402_1005Metric" V 6530 4850 50  0001 C CNN
 F 3 "~" H 6600 4850 50  0001 C CNN
 	1    6600 4850
@@
 F 0 "D1" V 6636 4232 50  0000 R CNN
 F 1 "LED" V 6546 4232 50  0000 R CNN
-F 2 "" H 6600 4350 50  0001 C CNN
+F 2 "LED_SMD:LED_0603_1608Metric" H 6600 4350 50  0001 C CNN
 F 3 "~" H 6600 4350 50  0001 C CNN
 	1    6600 4350
@@
 F 0 "R11" H 7070 4895 50  0000 L CNN
 F 1 "470" H 7070 4805 50  0000 L CNN
-F 2 "" V 6930 4850 50  0001 C CNN
+F 2 "Resistor_SMD:R_0402_1005Metric" V 6930 4850 50  0001 C CNN
 F 3 "~" H 7000 4850 50  0001 C CNN
 	1    7000 4850
@@
 F 0 "SW1" V 6755 5498 50  0000 L CNN
 F 1 "KEY_RST" V 6845 5498 50  0000 L CNN
-F 2 "" H 6800 5400 50  0001 C CNN
+F 2 "Button_Switch_SMD:SW_SPST_PTS810" H 6800 5400 50  0001 C CNN
 F 3 "" H 6800 5400 50  0001 C CNN
 	1    6800 5400
@@
 F 0 "R12" H 7870 4695 50  0000 L CNN
 F 1 "470" H 7870 4605 50  0000 L CNN
-F 2 "" V 7730 4650 50  0001 C CNN
+F 2 "Resistor_SMD:R_0402_1005Metric" V 7730 4650 50  0001 C CNN
 F 3 "~" H 7800 4650 50  0001 C CNN
 	1    7800 4650
@@
 F 0 "SW2" V 7800 4900 50  0000 L CNN
 F 1 "KEY_FLASH" H 7600 5250 50  0000 L CNN
-F 2 "" H 7800 5100 50  0001 C CNN
+F 2 "Button_Switch_SMD:SW_SPST_PTS810" H 7800 5100 50  0001 C CNN
 F 3 "" H 7800 5100 50  0001 C CNN
 	1    7800 5100
@@
 F 0 "R13" H 9870 4795 50  0000 L CNN
 F 1 "220k (1%)" H 9870 4705 50  0000 L CNN
-F 2 "" V 9730 4750 50  0001 C CNN
+F 2 "Resistor_SMD:R_0402_1005Metric" V 9730 4750 50  0001 C CNN
 F 3 "~" H 9800 4750 50  0001 C CNN
 	1    9800 4750
@@
 F 0 "R14" H 9870 5295 50  0000 L CNN
 F 1 "100k (1%)" H 9870 5205 50  0000 L CNN
-F 2 "" V 9730 5250 50  0001 C CNN
+F 2 "Resistor_SMD:R_0402_1005Metric" V 9730 5250 50  0001 C CNN
 F 3 "~" H 9800 5250 50  0001 C CNN
 	1    9800 5250
